File: hardware/BLV_Cutaway/BLV_Cutaway.kicad_sch (KiCad schematic)
At the start: 0 parts

Commit message: Created sheets for RF, MCU, Sensors, and Power.
Other:
- added sheet MCU (mcu.kicad_sch)
- added sheet Power (power.kicad_sch)
- added sheet RF (rf.kicad_sch)
- added sheet Sensors (sensors.kicad_sch)
- company: (none) -> Bronco S.T.A.R.
- title: (none) -> BLV Cutaway
Changed lines of the file:
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@@
 	(generator_version "10.0")
 	(paper "A4")
+	(title_block
+		(title "BLV Cutaway")
+		(date "2026-10-29")
+		(rev "1")
+		(company "Bronco S.T.A.R.")
+	)
+	(sheet
+		(at 101.6 50.8)
+		(size 50.8 50.8)
+		(exclude_from_sim no)
+		(in_bom yes)
+		(on_board yes)
+		(dnp no)
+		(fields_autoplaced yes)
+		(stroke
+			(width 0.1524)
+			(type solid)
+		)
+		(fill
+			(color 0 0 0 0)
+		)
+		(property "Sheetname" "MCU"
+			(at 101.6 50.0884 0)
+			(show_name no)
+			(do_not_autoplace no)
+			(effects
+				(font
+					(size 1.27 1.27)
+				)
+				(justify left bottom)
+			)
+		)
+		(property "Sheetfile" "mcu.kicad_sch"
+			(at 101.6 102.1846 0)
+			(show_name no)
+			(do_not_autoplace no)
+			(effects
+				(font
+					(size 1.27 1.27)
+				)
+				(justify left top)
+			)
+		)
+		(instances
+			(project "BLV_Cutaway"
+				(path "/80a23bfb-aae0-4207-bdfe-0eafbda2f7c7"
+					(page "2")
+				)
+			)
+		)
+	)
+	(sheet
+		(at 51.562 50.8)
+		(size 25.4 25.4)
+		(exclude_from_sim no)
+		(in_bom yes)
+		(on_board yes)
+		(dnp no)
+		(fields_autoplaced yes)
+		(stroke
+			(width 0.1524)
+			(type solid)
+		)
+		(fill
+			(color 0 0 0 0)
+		)
+		(property "Sheetname" "Sensors"
+			(at 51.562 50.0884 0)
+			(show_name no)
+			(do_not_autoplace no)
+			(effects
+				(font
+					(size 1.27 1.27)
+				)
+				(justify left bottom)
+			)
+		)
+		(property "Sheetfile" "sensors.kicad_sch"
+			(at 51.562 76.7846 0)
+			(show_name no)
+			(do_not_autoplace no)
+			(effects
+				(font
+					(size 1.27 1.27)
+				)
+				(justify left top)
+			)
+		)
+		(instances
+			(project "BLV_Cutaway"
+				(path "/80a23bfb-aae0-4207-bdfe-0eafbda2f7c7"
+					(page "5")
+				)
+			)
+		)
+	)
+	(sheet
+		(at 177.8 35.56)
+		(size 25.4 25.4)
+		(exclude_from_sim no)
+		(in_bom yes)
+		(on_board yes)
+		(dnp no)
+		(fields_autoplaced yes)
+		(stroke
+			(width 0.1524)
+			(type solid)
+		)
+		(fill
+			(color 0 0 0 0)
+		)
+		(property "Sheetname" "Power"
+			(at 177.8 34.8484 0)
+			(show_name no)
+			(do_not_autoplace no)
+			(effects
+				(font
+					(size 1.27 1.27)
+				)
+				(justify left bottom)
+			)
+		)
+		(property "Sheetfile" "power.kicad_sch"
+			(at 177.8 61.5446 0)
+			(show_name no)
+			(do_not_autoplace no)
+			(effects
+				(font
+					(size 1.27 1.27)
+				)
+				(justify left top)
+			)
+		)
+		(instances
+			(project "BLV_Cutaway"
+				(path "/80a23bfb-aae0-4207-bdfe-0eafbda2f7c7"
+					(page "3")
+				)
+			)
+		)
+	)
+	(sheet
+		(at 177.8 86.36)
+		(size 25.4 25.4)
+		(exclude_from_sim no)
+		(in_bom yes)
+		(on_board yes)
+		(dnp no)
+		(fields_autoplaced yes)
+		(stroke
+			(width 0.1524)
+			(type solid)
+		)
+		(fill
+			(color 0 0 0 0)
+		)
+		(property "Sheetname" "RF"
+			(at 177.8 85.6484 0)
+			(show_name no)
+			(do_not_autoplace no)
+			(effects
+				(font
+					(size 1.27 1.27)
+				)
+				(justify left bottom)
+			)
+		)
+		(property "Sheetfile" "rf.kicad_sch"
+			(at 177.8 112.3446 0)
+			(show_name no)
+			(do_not_autoplace no)
+			(effects
+				(font
+					(size 1.27 1.27)
+				)
+				(justify left top)
+			)
+		)
+		(instances
+			(project "BLV_Cutaway"
+				(path "/80a23bfb-aae0-4207-bdfe-0eafbda2f7c7"
+					(page "4")
+				)
+			)
+		)
+	)
 	(sheet_instances
 		(path "/"
